File: KDT_Hierarchical_KiBot.kicad_pcb (KiCad board)
At the start: 6 copper layers, 0 parts

Commit message: Add Edge.Cuts outline to example PCB
The interactive BoM tool (iBoM 2.11.2 in the KiCad 10 image) requires a
board outline on Edge.Cuts. The example board had none, failing the BoM
step. Added a rectangular outline enclosing the demo content.
Other:
- board outline added: 210 x 140 mm
Changed lines of the file:
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@@
 	(net 0 "")
+	(gr_rect
+		(start 10 15)
+		(end 220 155)
+		(stroke
+			(width 0.1)
+			(type default)
+		)
+		(fill none)
+		(layer "Edge.Cuts")
+	)
 	(gr_rect
 		(start 172 48.5)
